File: new_esplay.sch (EAGLE design)
At the start: 93 parts, among them J3 AUDIO_JACK_3.5MM_KIT, Q1 1.1A/60V/600mΩ, T1 2n2222, T2 2n2222, T3 2n2222, U2 MIC5219 3.3V

Commit message: Optimize vias and add amplifier
Parts:
- added C18: 47uF, SparkFun-Capacitors:47UF-POLAR-EIA3528-10V-10%
- added C19: 10uF, SparkFun-Capacitors:2.2UF-0805-25V-(+80/-20%)
- added C20: 0.01uF, SparkFun-Capacitors:2.2UF-0805-25V-(+80/-20%)
- added C21, C24: 0.1uF, SparkFun-Capacitors:2.2UF-0805-25V-(+80/-20%)
- added R38, R41: 4,7, SparkFun-Resistors:0.22OHM-0805-1/4W-1%
- added R39, R40: 100, SparkFun-Resistors:0.3OHM-0805-1/8W-1%
- added SPK+, SPK-: (no value), wirepad:SMD2
- added U1: TDA2822MSOIC8, TDA2822M:TDA2822MSOIC8
- S10, S12, S3, S4, S5, S6, S7, S8, S9: value MOMENTARY-SWITCH-SPST-SMD-5.2MM -> (none); device SparkFun-Switches:MOMENTARY-SWITCH-SPST-SMD-5.2MM -> SparkFun-Switches:MOMENTARY-SWITCH-SPST-2-SMD-5.2MM
Connections:
- new net N$15: J3.RSH, R39.1
- new net N$16: J3.TSH, R40.1
- new net N$17: R39.2, R40.2, U1.IN+(1)
- new net N$23: C19.2, C20.1, U1.IN-(2)
- new net N$30: C19.1, U1.IN-(1)
- new net N$31: C24.1, SPK+.P, U1.OUT_1
- new net N$32: C21.1, SPK-.P, U1.OUT_2
- new net N$33: C21.2, R38.1
- new net N$34: C24.2, R41.1
- net 3V3: now also C18.+, U1.SUPPLY_VOLTAGE
- net A: now also S9.3; no longer S9.2
- net B: now also S10.3; no longer S10.2
- net DOWN: now also S4.3; no longer S4.2
- net GND: now also C18.-, C20.2, ESP32-WROVER.EXP, J1.SHIELD, R38.2, R41.2, S10.2, S12.3, S12.4, S3.2, S4.2, S5.2, S6.2, S7.2, S8.2, S9.2, U1.GND, U1.IN+(2); no longer S12.2
- net LEFT: now also S5.3; no longer S5.2
- net RIGHT: now also S6.3; no longer S6.2
- net SELECT: now also S8.3; no longer S8.2
- net START: now also S7.3; no longer S7.2
- net UP: now also S3.3; no longer S3.2
Other:
- moved on the sheet: J3
