File: docs/new_esplay.brd (EAGLE design)
At the start: 100 x 50 mm, 118 parts, among them J1 MICROSD-PUSH-OUT, J5 AUDIO_JACK_3.5MM_KIT, Q1 1.1A/60V/600mΩ, T1 2n2222, T2 2n2222, T3 2n2222, U1 PCF8574, U2 MIC5219 3.3V, U3 LTC4054LES5-4.2#TRPBF, U4 CH340C/G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

Commit message: final design rev2.0
Parts:
- C1, C4, C8, C9: value 0.1uF -> 100nF
- C10, C12, C14, C15, C16, C17, C21, C22, C23, C24, C25, C26, C5: device PP_Passives:0805 -> SparkFun-Capacitors:0805
- C20: value 0.1uF -> 100nF; device PP_Passives:0805 -> SparkFun-Capacitors:0805
- C6: value 470pf -> 470pF
- J5: value AUDIO_JACK_3.5MM_KIT -> AUDIO_JACK_3.5MM_PTH; device SparkFun-Connectors:AUDIO-JACK-KIT -> SparkFun-Connectors:AUDIO-JACK
- R17, R26: value 100k -> 100K
- R23: value 10k -> 10K
- R37: value 1 -> 1K
- T1, T2, T3: value 2n2222 -> 600mA/40V; device zetex:SOT-23 -> SparkFun-DiscreteSemi:SOT23-3
- U4: value CH340C/G -> CH340G
- moved T1 0.18 mm to (35.6, 23.6), turned to 180 degrees
- turned T2 to 180 degrees
- turned T3 to 180 degrees
Connections:
- net DTR: now also T2.3; no longer T2.1
- net LCD_BCKL: now also T3.1; no longer T3.3
- net N$12: now also T1.1; no longer T1.3
- net N$13: now also T2.1; no longer T2.3
- net N$9: now also T3.3; no longer T3.1
- net RESET: now also T1.3; no longer T1.1
Routing:
- net USB_DET: track 38.5 -> 33.1 mm, vias 0 -> 2
- net DOWN: track 26.4 -> 27.3 mm
- net SD_CLK: track 59.6 -> 60.3 mm
- net VIN: track 152.1 -> 152.7 mm

Commit message: bugs fix
Parts:
- R37: value 1K -> 1
- moved R38 1.20 mm to (86.0, 13.6)
- moved C17 1.05 mm to (81.3, 13.6)
- moved C22 1.02 mm to (89.2, 13.6)
- turned T2 to 0 degrees
Connections:
- net DTR: now also T2.2; no longer T2.3
- net IO0: now also T2.3; no longer T2.2
Routing:
- net RTS: track 20.1 -> 16.8 mm, vias 0 -> 2
- net N$13: track 2.65 -> 5.39 mm
- net N$30: track 4.85 -> 5.85 mm
- net DTR: track 16.7 -> 15.7 mm
- net N$14: track 37.9 -> 37.0 mm
- net N$23: track 2.03 -> 1.38 mm
- net N$16: track 4.10 -> 3.58 mm
- net GND: vias 17 -> 18
Other:
- board text added: "pcb-rev2.1-20190926"
- board text removed: "pcb-rev2.0-20190823"

Commit message: bugs fix with R19 value
Parts:
- R19: value 100 -> 10
Changed lines of the file:
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@@
 <drawing>
 <settings>
-<setting alwaysvectorfont="yes"/>
+<setting alwaysvectorfont="no"/>
 <setting verticaltext="up"/>
 </settings>
@@
 <attribute name="VALUE" x="11.43" y="34.671" size="0.6096" layer="28" font="vector" ratio="20" rot="MR0" align="top-center"/>
 </element>
-<element name="R19" library="SparkFun-Resistors" library_urn="urn:adsk.eagle:library:12877214" package="0805" package3d_urn="urn:adsk.eagle:package:12877276/2" value="100" x="63.5" y="27.94" smashed="yes" rot="MR270">
+<element name="R19" library="SparkFun-Resistors" library_urn="urn:adsk.eagle:library:12877214" package="0805" package3d_urn="urn:adsk.eagle:package:12877276/2" value="10" x="63.5" y="27.94" smashed="yes" rot="MR270">
 <attribute name="NAME" x="61.849" y="27.94" size="0.8128" layer="26" font="vector" ratio="20" rot="MR270" align="bottom-center"/>
 <attribute name="PROD_ID" value="RES-09883" x="154.94" y="-36.83" size="1.778" layer="28" rot="MR270" display="off"/>
