File: docs/new_esplay.sch (EAGLE design)
At the start: 115 parts, among them J1 MICROSD-PUSH-OUT, J5 AUDIO_JACK_3.5MM_KIT, Q1 1.1A/60V/600mΩ, T1 2n2222, T2 2n2222, T3 2n2222, U1 PCF8574, U2 MIC5219 3.3V, U3 LTC4054LES5-4.2#TRPBF, U4 CH340C/G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

Commit message: final design rev2.0
Parts:
- C1, C4, C8, C9: value 0.1uF -> 100nF
- C10, C12, C14, C15, C16, C17, C21, C22, C23, C24, C25, C26, C5: device PP_Passives:CAPACITOR_NON_POLAR_0805 -> SparkFun-Capacitors:2.2UF-0805-25V-(+80/-20%)
- C20: value 0.1uF -> 100nF; device PP_Passives:CAPACITOR_NON_POLAR_0805 -> SparkFun-Capacitors:2.2UF-0805-25V-(+80/-20%)
- C6: value 470pf -> 470pF
- J5: value AUDIO_JACK_3.5MM_KIT -> AUDIO_JACK_3.5MM_PTH; device SparkFun-Connectors:AUDIO_JACK_3.5MM_KIT -> SparkFun-Connectors:AUDIO_JACK_3.5MM_PTH
- R17, R26: value 100k -> 100K
- R23: value 10k -> 10K
- R37: value 1 -> 1K
- T1, T2, T3: value 2n2222 -> 600mA/40V; device zetex:NPNSOT23 -> SparkFun-DiscreteSemi:TRANS_NPN-MMBT2222AL
- U4: value CH340C/G -> CH340G
Other:
- moved on the sheet: C10, C11, C12, C14, C15, C16, C17, C20, C21, C22, C23, C24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

Commit message: bugs fix
Parts:
- R37: value 1K -> 1
Connections:
- net DTR: now also T2.E; no longer T2.C
- net IO0: now also T2.C; no longer T2.E
Other:
- moved on the sheet: T2
Changed lines of the file:
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@@
 <part name="FRAME1" library="SparkFun-Aesthetics" library_urn="urn:adsk.eagle:library:12892397" deviceset="FRAME-A4L" device="">
 <attribute name="CNAME" value="ESPLAY MICRO"/>
-<attribute name="CREVISION" value="2.0"/>
+<attribute name="CREVISION" value="2.1"/>
 <attribute name="DESIGNER" value="FUJI PEBRI"/>
 </part>
 <part name="FRAME2" library="SparkFun-Aesthetics" library_urn="urn:adsk.eagle:library:12892397" deviceset="FRAME-A4L" device="">
 <attribute name="CNAME" value="ESPLAY MICRO"/>
-<attribute name="CREVISION" value="2.0"/>
+<attribute name="CREVISION" value="2.1"/>
 <attribute name="DESIGNER" value="FUJI PEBRI"/>
 </part>
@@
 <part name="R40" library="SparkFun-Resistors" library_urn="urn:adsk.eagle:library:12877214" deviceset="0.3OHM" device="-0805-1/8W-1%" package3d_urn="urn:adsk.eagle:package:12877276/2" value="220K"/>
 <part name="R32" library="SparkFun-Resistors" library_urn="urn:adsk.eagle:library:12877214" deviceset="0.3OHM" device="-0805-1/8W-1%" package3d_urn="urn:adsk.eagle:package:12877276/2" value="1"/>
-<part name="R37" library="SparkFun-Resistors" library_urn="urn:adsk.eagle:library:12877214" deviceset="0.3OHM" device="-0805-1/8W-1%" package3d_urn="urn:adsk.eagle:package:12877276/2" value="1K"/>
+<part name="R37" library="SparkFun-Resistors" library_urn="urn:adsk.eagle:library:12877214" deviceset="0.3OHM" device="-0805-1/8W-1%" package3d_urn="urn:adsk.eagle:package:12877276/2" value="1"/>
 <part name="GND34" library="SparkFun-PowerSymbols" deviceset="GND" device=""/>
 <part name="GND31" library="SparkFun-PowerSymbols" deviceset="GND" device=""/>
@@
 <attribute name="VALUE" x="170.18" y="160.02" size="1.778" layer="96"/>
 </instance>
-<instance part="T2" gate="G$1" x="165.1" y="147.32" smashed="yes">
-<attribute name="NAME" x="170.18" y="147.32" size="1.778" layer="95"/>
-<attribute name="VALUE" x="170.18" y="144.78" size="1.778" layer="96"/>
+<instance part="T2" gate="G$1" x="165.1" y="147.32" smashed="yes" rot="MR180">
+<attribute name="NAME" x="170.18" y="147.32" size="1.778" layer="95" rot="MR180"/>
+<attribute name="VALUE" x="170.18" y="149.86" size="1.778" layer="96" rot="MR180"/>
 </instance>
 <instance part="R8" gate="G$1" x="149.86" y="162.56" smashed="yes" rot="R180">
@@
 </segment>
 <segment>
-<pinref part="T2" gate="G$1" pin="E"/>
-<wire x1="167.64" y1="142.24" x2="172.72" y2="142.24" width="0.1524" layer="91"/>
-<label x="172.72" y="142.24" size="1.27" layer="95" xref="yes"/>
-</segment>
-<segment>
 <pinref part="JP1" gate="G$1" pin="2"/>
 <wire x1="106.68" y1="66.04" x2="109.22" y2="66.04" width="0.1524" layer="91"/>
 <label x="109.22" y="66.04" size="1.27" layer="95" xref="yes"/>
+</segment>
+<segment>
+<pinref part="T2" gate="G$1" pin="C"/>
+<wire x1="167.64" y1="142.24" x2="172.72" y2="142.24" width="0.1524" layer="91"/>
+<label x="172.72" y="142.24" size="1.27" layer="95" xref="yes"/>
 </segment>
 </net>
@@
 <wire x1="139.7" y1="162.56" x2="139.7" y2="152.4" width="0.1524" layer="91"/>
 <junction x="139.7" y="162.56"/>
-<pinref part="T2" gate="G$1" pin="C"/>
+<label x="137.16" y="162.56" size="1.27" layer="95" rot="R180" xref="yes"/>
+<pinref part="T2" gate="G$1" pin="E"/>
 <wire x1="139.7" y1="152.4" x2="167.64" y2="152.4" width="0.1524" layer="91"/>
-<label x="137.16" y="162.56" size="1.27" layer="95" rot="R180" xref="yes"/>
-</segment>
-</net>
+</segment>
+</net>

Commit message: bugs fix with R19 value
Parts:
- R19: value 100 -> 10
Changed lines of the file:
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@@
 <part name="GND16" library="supply1" library_urn="urn:adsk.eagle:library:371" deviceset="GND" device=""/>
 <part name="T3" library="SparkFun-DiscreteSemi" library_urn="urn:adsk.eagle:library:12892623" deviceset="TRANS_NPN" device="-MMBT2222AL" package3d_urn="urn:adsk.eagle:package:12892688/2" value="600mA/40V"/>
-<part name="R19" library="SparkFun-Resistors" library_urn="urn:adsk.eagle:library:12877214" deviceset="0.22OHM" device="-0805-1/4W-1%" package3d_urn="urn:adsk.eagle:package:12877276/2" value="100"/>
+<part name="R19" library="SparkFun-Resistors" library_urn="urn:adsk.eagle:library:12877214" deviceset="0.22OHM" device="-0805-1/4W-1%" package3d_urn="urn:adsk.eagle:package:12877276/2" value="10"/>
 <part name="R17" library="SparkFun-Resistors" library_urn="urn:adsk.eagle:library:12877214" deviceset="0.22OHM" device="-0805-1/4W-1%" package3d_urn="urn:adsk.eagle:package:12877276/2" value="100K"/>
 <part name="GND14" library="supply1" library_urn="urn:adsk.eagle:library:371" deviceset="GND" device=""/>
